Commit message: Add per-serial mesh-frame optical/depth TF and depth-frame publishers
- digit.xacro: add tactile_<serial>_mesh_frame mirroring the visual origin
  rotation; define tactile_<serial>_optical_frame (vendor finger_pose frame)
  and tactile_<serial>_depth_frame as fixed children in mesh-frame coordinates.
- raw/surface/force publishers: publish in tactile_<serial>_depth_frame.
- multi_sensor_tactile_streamer: remove YAML-driven optical static TF.
- sensor YAMLs: remove optical_frame blocks (now hardcoded in xacro).
- update digit.stl mesh asset.

File: ros2/urdf/digit.xacro (robot description, xacro)
@@ -2,5 +2,10 @@
 <xacro:macro name="digit_sensor"
              params="serial">
-  <!-- DIGIT sensor body (realsense-style: mesh origin hardcoded, optical frame offset from driver YAML) -->
+  <!-- DIGIT sensor body: mesh origin hardcoded; optical and depth frames are
+       fixed joints defined here. Depth frame is the camera frame used by
+       depth/pointcloud publishers; optical frame is the vendor finger_pose
+       matching frame. Offsets are w.r.t. the digit mesh frame, so they are
+       parented to tactile_${serial}_mesh_frame, which mirrors the visual
+       origin rotation applied to the STL mesh. -->
   <link name="tactile_${serial}_base_link">
     <visual>
@@ -26,6 +31,24 @@
                iyx="0.0000000e+00" iyy="3.8502616e-06" iyz="0.0000000e+00"
                izx="0.0000000e+00" izy="0.0000000e+00" izz="3.8502616e-06"/>
-    </inertial>
+      </inertial>
   </link>
+  <link name="tactile_${serial}_mesh_frame"/>
+  <joint name="mesh_${serial}" type="fixed">
+    <parent link="tactile_${serial}_base_link"/>
+    <child link="tactile_${serial}_mesh_frame"/>
+    <origin rpy="1.5708 0 1.5708" xyz="0 0 0"/>
+  </joint>
+  <link name="tactile_${serial}_optical_frame"/>
+  <joint name="optical_${serial}" type="fixed">
+    <parent link="tactile_${serial}_mesh_frame"/>
+    <child link="tactile_${serial}_optical_frame"/>
+    <origin xyz="0.0 -0.004787 0.016802" rpy="0.01745329252 0.0 0.0"/>
+  </joint>
+  <link name="tactile_${serial}_depth_frame"/>
+  <joint name="depth_optical_${serial}" type="fixed">
+    <parent link="tactile_${serial}_mesh_frame"/>
+    <child link="tactile_${serial}_depth_frame"/>
+    <origin xyz="0.0 0.017475 0.017191" rpy="0.01745329252 0.0 0.0"/>
+  </joint>
 </xacro:macro>
 </robot>

Commit message: Remove per-sensor mesh_frame TF; parent optical/depth frames to base_link

File: ros2/urdf/digit.xacro (robot description, xacro)
@@ -5,7 +5,7 @@
        fixed joints defined here. Depth frame is the camera frame used by
        depth/pointcloud publishers; optical frame is the vendor finger_pose
-       matching frame. Offsets are w.r.t. the digit mesh frame, so they are
-       parented to tactile_${serial}_mesh_frame, which mirrors the visual
-       origin rotation applied to the STL mesh. -->
+       matching frame. Offsets are composed base-frame values, so optical and
+       depth are parented directly to tactile_${serial}_base_link; the empty
+       mesh_frame TF parent is removed. -->
   <link name="tactile_${serial}_base_link">
     <visual>
@@ -33,21 +33,15 @@
       </inertial>
   </link>
-  <link name="tactile_${serial}_mesh_frame"/>
-  <joint name="mesh_${serial}" type="fixed">
-    <parent link="tactile_${serial}_base_link"/>
-    <child link="tactile_${serial}_mesh_frame"/>
-    <origin rpy="1.5708 0 1.5708" xyz="0 0 0"/>
-  </joint>
   <link name="tactile_${serial}_optical_frame"/>
   <joint name="optical_${serial}" type="fixed">
-    <parent link="tactile_${serial}_mesh_frame"/>
+    <parent link="tactile_${serial}_base_link"/>
     <child link="tactile_${serial}_optical_frame"/>
-    <origin xyz="0.0 -0.004787 0.016802" rpy="0.01745329252 0.0 0.0"/>
+    <origin xyz="0.016802 0.0 -0.004787" rpy="1.588253 0.0 1.5708"/>
   </joint>
   <link name="tactile_${serial}_depth_frame"/>
   <joint name="depth_optical_${serial}" type="fixed">
-    <parent link="tactile_${serial}_mesh_frame"/>
+    <parent link="tactile_${serial}_base_link"/>
     <child link="tactile_${serial}_depth_frame"/>
-    <origin xyz="0.0 0.017475 0.017191" rpy="0.01745329252 0.0 0.0"/>
+    <origin xyz="0.017191 0.0 0.017475" rpy="1.588253 0.0 1.5708"/>
   </joint>
 </xacro:macro>

Commit message: Align DIGIT optical/depth frames to REP-103 z-forward

File: ros2/urdf/digit.xacro (robot description, xacro)
@@ -37,5 +37,8 @@
     <parent link="tactile_${serial}_base_link"/>
     <child link="tactile_${serial}_optical_frame"/>
-    <origin xyz="0.016802 0.0 -0.004787" rpy="1.588253 0.0 1.5708"/>
+    <!-- +Z forward (REP-103 optical): measured base orientation (1.588253, 0, 1.5708)
+         rotated exactly -90deg about X -> (0.0175, 0, 1.5708), then -90deg about Z
+         to align image axes with depth_frame -> (0, 0.0175, 0) -->
+    <origin xyz="0.016802 0.0 -0.004787" rpy="0.0 0.0175 0.0"/>
   </joint>
   <link name="tactile_${serial}_depth_frame"/>
@@ -43,5 +46,7 @@
     <parent link="tactile_${serial}_base_link"/>
     <child link="tactile_${serial}_depth_frame"/>
-    <origin xyz="0.017191 0.0 0.017475" rpy="1.588253 0.0 1.5708"/>
+    <!-- Depth/PC frame: +Z forward (REP-103), image roll corrected by -90deg
+         about Z in the +Z-forward frame -> (0, 0.0175, 0) -->
+    <origin xyz="0.017191 0.0 0.017475" rpy="0.0 0.0175 0.0"/>
   </joint>
 </xacro:macro>
